Commit message: feat:add dynamic model

File: src/asr_sdm_universe/robot/asr_sdm_description/urdf/underwater_snakerobot.urdf (robot description, URDF)
Before this commit: robot underwater_snakerobot_description, 6 links, 5 joints
Links:
- added link joint1_intermediate, mass 0.001; visual sphere radius=0.035
- added link joint2_intermediate, mass 0.001; visual sphere radius=0.035
- added link joint3_intermediate, mass 0.001; visual sphere radius=0.035
- added link link_3, mass 2.0; collision cylinder length=0.3 radius=0.06; visual cylinder length=0.3 radius=0.06
- added link link_4, mass 2.0; collision cylinder length=0.3 radius=0.06; visual cylinder length=0.3 radius=0.06
- added link screw_3_left; visual mesh filename=package://asr_sdm_description/meshes/screw_left_CFD.dae
- added link screw_3_right; visual mesh filename=package://asr_sdm_description/meshes/screw_right_CFD.dae
- added link screw_4_left; visual mesh filename=package://asr_sdm_description/meshes/screw_left_CFD.dae
- added link screw_4_right; visual mesh filename=package://asr_sdm_description/meshes/screw_right_CFD.dae
- link base_link: mass 2 -> 2.0; geometry collision cylinder length=0.3 radius=0.06; visual cylinder length=0.10 radius=0.06
- link link_2: mass 2 -> 2.0; geometry collision cylinder length=0.3 radius=0.06; visual cylinder length=0.3 radius=0.06
- link screw_1_left: geometry visual mesh filename=package://asr_sdm_description/meshes/screw_left_CFD.dae
Joints:
- removed joint base_link_to_link_2
- removed joint base_link_to_screw_1_left_joint
- removed joint base_link_to_screw_1_right_joint
- removed joint link_2_to_screw_2_left_joint
- removed joint link_2_to_screw_2_right_joint
- added joint joint1_pitch: type revolute, parent base_link, child joint1_intermediate, origin xyz=-0.15 0 0 rpy=0 0 0, axis 0 1 0, limit lower=-1.57 upper=1.57 effort=100.0 velocity=10.0
- added joint joint1_yaw: type revolute, parent joint1_intermediate, child link_2, origin xyz=-0.15 0 0 rpy=0 0 0, axis 0 0 1, limit lower=-1.57 upper=1.57 effort=100.0 velocity=10.0
- added joint joint2_pitch: type revolute, parent link_2, child joint2_intermediate, origin xyz=-0.15 0 0 rpy=0 0 0, axis 0 1 0, limit lower=-1.57 upper=1.57 effort=100.0 velocity=10.0
- added joint joint2_yaw: type revolute, parent joint2_intermediate, child link_3, origin xyz=-0.15 0 0 rpy=0 0 0, axis 0 0 1, limit lower=-1.57 upper=1.57 effort=100.0 velocity=10.0
- added joint joint3_pitch: type revolute, parent link_3, child joint3_intermediate, origin xyz=-0.15 0 0 rpy=0 0 0, axis 0 1 0, limit lower=-1.57 upper=1.57 effort=100.0 velocity=10.0
- added joint joint3_yaw: type revolute, parent joint3_intermediate, child link_4, origin xyz=-0.15 0 0 rpy=0 0 0, axis 0 0 1, limit lower=-1.57 upper=1.57 effort=100.0 velocity=10.0
- added joint link1_to_screw_1_left: type continuous, parent base_link, child screw_1_left, origin xyz=0.10 0.07 0 rpy=0 0 0, axis 1 0 0
- added joint link1_to_screw_1_right: type continuous, parent base_link, child screw_1_right, origin xyz=0.10 -0.07 0 rpy=0 0 0, axis 1 0 0
- added joint link2_to_screw_2_left: type continuous, parent link_2, child screw_2_left, origin xyz=0.10 0.07 0 rpy=0 0 0, axis 1 0 0
- added joint link2_to_screw_2_right: type continuous, parent link_2, child screw_2_right, origin xyz=0.10 -0.07 0 rpy=0 0 0, axis 1 0 0
- added joint link3_to_screw_3_left: type continuous, parent link_3, child screw_3_left, origin xyz=0.10 0.07 0 rpy=0 0 0, axis 1 0 0
- added joint link3_to_screw_3_right: type continuous, parent link_3, child screw_3_right, origin xyz=0.10 -0.07 0 rpy=0 0 0, axis 1 0 0
- added joint link4_to_screw_4_left: type continuous, parent link_4, child screw_4_left, origin xyz=0.10 0.07 0 rpy=0 0 0, axis 1 0 0
- added joint link4_to_screw_4_right: type continuous, parent link_4, child screw_4_right, origin xyz=0.10 -0.07 0 rpy=0 0 0, axis 1 0 0
